File: out/earring.kicad_sch (KiCad schematic)
At the start: 123 parts, among them J1 USB-C, SW1 BOOTSEL, SW2 PWR, U1 RP2350A, U2 LGS4056H, U3 NCP730-3.3, U4 TPS22913, U5 USBLC6-2P6, U6 LSM6DS3TR-C, U7 W25Q16JVUXIQ, Y1 12MHz

Commit message: Rev 2 power path: split VBATT from VSYS so USB runs the board
Rev 1 hung the LDO input and the LED load switch on VBATT -- the same
node as the charger's BAT pin -- so the LGS4056H's ~41mA program current
was SHARED with the running system. 17mA of MCU plus 17.5mA of LED rail
left the cell about 6mA, and a flat cell could never climb to the
SK6805-EC10's 3.7V minimum VDD before someone unplugged it. That is the
"no lights at all" failure from Aug 27, and it is a power-path problem,
not a firmware one.

  VBUS  --|>|--  VSYS      D3, B5819WS Schottky, ~0.3V at our ~60mA
  VBATT --[Q2]-- VSYS      CJ2101 P-FET, on only when no cable is in
  VSYS  -> U3 (LDO IN), U4 (LED load switch IN), C18, C29
  VBATT -> U2 pin 5 (charger BAT), BT1, C17, SW2   [cell node ONLY]

Q2's ORIENTATION IS THE WHOLE TRICK: source = VSYS, drain = VBATT. A
P-FET's body diode conducts drain->source, so this way it points
cell->VSYS. It blocks the 4.7V USB rail from back-feeding the cell
around the charger -- which is exactly what the intuitive wiring
(source on the battery) would do through the body diode -- while still
letting the cell carry the load through ~0.4V of diode if VSYS sags
below VBATT, covering the ~200ms of VBUS decay on unplug. Gate is
R22 10k from VBUS against R21 1M to GND: near VBUS with a cable in
(Vgs +0.25V, hard off), and following the dead VBUS node without one.
That node is not floating -- R19/R20 pin it under 0.65V even against
R18's backfeed -- so Vgs is -2.4V at a 3.0V cell and Q2 is fully on.

This retires the R8 22k->15k rework rather than performing it. 22k
already gives 40.9mA, which is exactly the fitted RJD2032C1's rated
40mA charge, and the reason 15k was tempting is gone. The hazard that
blocked it is gone too: with the system off the cell, the full program
current reaches the cell in EITHER switch position.

What else falls out: DONE can finally assert (the cell's current
actually tapers to ITERM now), VBSENSE reads a true unloaded cell while
charging, the r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
Parts:
- added C26: 100n, earring:C_0402_1005Metric, symbol gen:C
- added C29: 10u, earring:C_0603_1608Metric, symbol gen:C
- added D2: BAT54S, earring:SOT-323_BAT54SW, symbol gen:D_SS
- added D3: B5819WS, earring:D_SOD-323, symbol gen:D_SCH
- added Q1: ALS-PT19, earring:SENSOR_ALS-PT19, symbol gen:light_sensor
- added Q2: CJ2101, earring:SOT-323_MOSFET, symbol gen:Q_PMOS
- added Q3: BSS138W, earring:SOT-323_MOSFET, symbol gen:Q_NMOS
- added R16: 22k, earring:R_0402_1005Metric, symbol gen:R
- added R17, R18: 100k, earring:R_0402_1005Metric, symbol gen:R
- added R19, R20, R22: 10k, earring:R_0402_1005Metric, symbol gen:R
- added R21: 1M, earring:R_0402_1005Metric, symbol gen:R
- added R23: 1k, earring:R_0402_1005Metric, symbol gen:R
- BT1: footprint earring:BAT_CR2032_W -> earring:BAT_MY2032_12R
Connections:
- net 3V3: now also Q1.1 (C)
- net GND: now also C26.2, C29.2, Q3.2 (S), R16.2, R17.2, R20.2, R21.2
- net LED_D0: now also Q3.3 (D), R23.2; no longer U1.29 (GPIO18)
- net PWR_EN: now also D2.3 (K1A2), R17.1, R18.2; no longer SW2.2
- net VBATT: now also D2.2 (K2), Q2.3 (D); no longer C18.1, R11.1, U3.6 (IN), U4.A2 (VIN)
- net VBUS: now also D3.2 (A), R18.1, R19.1, R22.1
- net VLED: now also R23.1
- net LIGHT: now reaches U1.40 (GPIO26/ADC0)
- net LIGHT: now also C26.1, Q1.2 (E), R16.1
- net VBUS_SENSE: now reaches U1.41 (GPIO27)
- net VBUS_SENSE: now also R19.2, R20.1
- new net LED_DATA: Q3.1 (G), U1.29 (GPIO18)
- new net PATH_GATE: Q2.1 (G), R21.1, R22.2
- new net SW_ON: D2.1 (A1), R11.1, SW2.2
- new net VSYS: C18.1, C29.1, D3.1 (K), Q2.2 (S), U3.6 (IN), U4.A2 (VIN)
- no-connect marks 32 -> 30
Other:
- note added: "138 components / 87 nets / 4-layer JLCPCB stackup. Power rails (GND, 3V3, VBATT, VSYS, VLED, VBUS, VDD_CORE) are power symbols; only cross-block signals use global labels. Generated from scripts/circuit.py — do not hand-edit; rebuild with `python3 build.py --only schematic`."
- note added: "1M:1M divider off SW_ON, the switch common (rev 2 — was"
- note added: "3V3 LDO — EN = slide switch OR USB (diode-OR, clamped)"
- note added: "ALS-PT19 visible-light phototransistor; 22k"
- note added: "Ambient light sensor -> ADC0 (rev 2)"
- note added: "CHRG and DONE both release at termination, so they cannot tell 'unplugged' from 'plugged in and"
- note added: "LED data level shifter — open-drain into the ring"
- note added: "Rev 2: USB boots the board even with SW2 off. Against R17's"
- note added: "Rev 2: VBATT is the cell alone, VSYS runs the board, so the charger's whole 41mA reaches the cell in"
- note added: "Switch / battery sense -> ADC"
- note added: "Switch OFF + USB: reads 0, telling firmware to show"
- note added: "The ring's VIH is 0.7*VLED. On the cell that peaked at 2.94V and the MCU drove pixel 1"
- note added: "USB cable present — 10k:10k tap on VBUS -> ADC1"
- note added: "USB wake — VBUS feeds EN through R18"
- note added: "VBATT). Switch ON: VBATT/2 battery telemetry as before."
- note added: "charge status instead of running the show. GPIO29/ADC3."
- note added: "directly; on VSYS it is 3.29V (3.5V at a 5.25V port), past anything a 3.3V pad can"
- note added: "drain->source, so that way round it blocks USB from back-feeding the cell past the charger."
- note added: "either switch position. Q2's SOURCE is VSYS and its drain VBATT — a P-FET body diode conducts"
- note added: "full'. 10k:10k, not the 100k/1M used elsewhere: PWR_EN backfeeds through R18 and would float"
- note added: "it to VBATT+Vf (NCP730 abs max V_EN is VIN+0.3, even during"
- note added: "load -> ~0.33V @ 100 lux, saturates ~900"
- note added: "lux. Reads on GPIO26/ADC0."
- note added: "one). That is also what holds Q2's gate low enough to keep the battery path on."
- note added: "output. Q3 inverts into R23's pull-up, so the swing is a full VLED rail whatever VLED is"
- note added: "override sits after the PIO, so the NeoPixel program is untouched."
- note added: "power path — VBUS runs the board when a cable is in"
- note added: "precharge of a dead cell). Firmware then sees SW_ON=0 on"
- note added: "previous DO. Firmware must set gpio_set_outover(LED_DATA, GPIO_OVERRIDE_INVERT) — the pad"
- note added: "pulldown EN sits at ~VBUS/2, and D2's second diode clamps"
- note added: "running the show."
- note added: "the sense divider and shows charge status instead of"
- note added: "this node high, so the tap has to be stiff enough to swamp it (0.33V no cable, 2.2-2.75V with"
- note added: "— 3.0V cell or 5.0V cable. Only pixel 1 needs it; every DI after that is driven by the"
- note removed: "123 components / 81 nets / 4-layer JLCPCB stackup. Power rails (GND, 3V3, VBATT, VLED, VBUS, VDD_CORE) are power symbols; only cross-block signals use global labels. Generated from scripts/circuit.py — do not hand-edit; rebuild with `python3 build.py --only schematic`."
- note removed: "1M:1M divider -> half VBATT, filtered; read on"
- note removed: "3V3 LDO + power slide switch (switches EN, not the cell)"
- note removed: "Battery voltage sense -> ADC"
- note removed: "GPIO29/ADC3."
- moved on the sheet: C11, C12, C13, C14, C15, C20, C22, C25, C5, C6, L1, R1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

Commit message: Rev 2 coin-cell close-out: name the clip not the cell, BS-6 socket fit test
BT1's value is now the clip's MPN (MY-2032-12-R) so the BOM Comment agrees
with its LCSC column; design.yaml's power.battery is the one place the
hand-fitted RJD2032C1 cell is named. Adds the C22363833 (CR2032-BS-6) fit
study (scripts/gen_bs6_svg.py + dashboard entry): its land runs 1.19mm off
the board, and the only land-legal rotations put the body on J1.

Last commit of the coin-cell power source before the LiPo change.

Co-Authored-By: Claude Opus 5.5 <noreply@anthropic.com>
Parts:
- BT1: value LIR2032 -> MY-2032-12-R
Other:
- note added: "Li-ion charger (LGS4056H, ~41mA) + RJD2032C1 cell"
- note removed: "Li-ion charger (LGS4056H, ~41mA) + LIR2032 cell"
Changed lines of the file:
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@@
 		(property "Reference" "BT1" (at 117.18 177.49 0)
 			(effects (font (size 1.27 1.27)) (justify left bottom)))
-		(property "Value" "LIR2032" (at 117.18 180.59 0)
+		(property "Value" "MY-2032-12-R" (at 117.18 180.59 0)
 			(effects (font (size 1.27 1.27)) (justify left bottom)))
 		(property "Footprint" "earring:BAT_MY2032_12R" (at 113.88 179.49 0)
@@
 		(stroke (width 0.1524) (type dash))
 )
-	(text "Li-ion charger (LGS4056H, ~41mA) + LIR2032 cell" (at 13.63 159.4 0)
+	(text "Li-ion charger (LGS4056H, ~41mA) + RJD2032C1 cell" (at 13.63 159.4 0)
 		(effects (font (size 2.2 2.2) (bold yes)) (justify left bottom))
 )
