File: out/earring.kicad_sch (KiCad schematic)
At the start: 138 parts, among them J1 USB-C, Q1 ALS-PT19, Q2 CJ2101, Q3 BSS138W, SW1 BOOTSEL, SW2 PWR, U1 RP2350A, U2 LGS4056H, U3 NCP730-3.3, U4 TPS22913, U5 USBLC6-2P6, U6 LSM6DS3TR-C, U7 W25Q16JVUXIQ, Y1 12MHz

Commit message: LiPo power source: LPR302823 on wire pads, B3U soft-latch power button
Replaces the RJD2032C1 coin cell + MY-2032-12-R clip with a LiPol
LPR302823 round pouch (Ø28 D-cut, 140 mAh) taped to the back and wired to
two pre-tinned pads beside J1. Placed and DRC-clean (0 errors), NOT routed:
routing is deferred to a new autorouter.

- BT1 -> BAT_LPR302823_PADS (no LCSC part). Pads sit >=0.6 mm from all
  other copper, and route.py keeps vias >=0.6 mm off them.
- R8 22k -> 18k (50 mA; cell max 70 mA). CV stays 4.20 V because the cell's
  PCM can trip as low as 4.305 V.
- SW2 slide switch -> Omron B3U-3000P side-push on the left tip edge, plus
  a CPU-held soft latch (Q4 CJ2101, Q5 BSS138W, D4 BAV70W, R24/R25, C27;
  GPIO20 PWR_HOLD, GPIO21 BTN_SENSE). The Ø28 cell covers the old switch
  spot at every legal angle. Firmware must now hold PWR_HOLD.
- route.py: the coin clip's via keepouts are gone (back centre now
  routable), and a polygon-accurate fallback is added for the tip-LED VLED
  via search.
- design/: intent, brief, decisions and gate evidence for phases 0/1/2/4/6,
  each with an independent review. Datasheets are in design/datasheets/.

The coin-cell rev 2 is commit 4538da2.

Co-Authored-By: Claude Opus 5.5 <noreply@anthropic.com>
Parts:
- added C27: 100n, earring:C_0402_1005Metric, symbol gen:C
- added D4: BAV70W, earring:SOT-323_BAT54SW, symbol gen:D_CC
- added Q4: CJ2101, earring:SOT-323_MOSFET, symbol gen:Q_PMOS_HS
- added Q5: BSS138W, earring:SOT-323_MOSFET, symbol gen:Q_NMOS
- added R24, R25: 100k, earring:R_0402_1005Metric, symbol gen:R
- BT1: value MY-2032-12-R -> LPR302823; footprint earring:BAT_MY2032_12R -> earring:BAT_LPR302823_PADS
- R8: value 22k -> 18k
- SW2: footprint earring:SW-TH_MSK12C02 -> earring:SW_B3U-3000P; symbol gen:SW_SPDT -> gen:SW_PUSH2
Connections:
- net GND: now also SW2.1, C27.2, Q5.2 (S), R25.2; no longer SW2.3
- net SW_ON: now also Q4.3 (D); no longer SW2.2
- net VBATT: now also Q4.2 (S), R24.1; no longer SW2.1
- net PWR_HOLD: now reaches U1.32 (GPIO20)
- net PWR_HOLD: now also Q5.1 (G), R25.1
- net BTN_SENSE: now reaches U1.33 (GPIO21)
- net BTN_SENSE: now also D4.1 (A1)
- new net BTN_N: C27.1, D4.3 (K), SW2.2
- new net LATCH_G: D4.2 (A2), Q4.1 (G), Q5.3 (D), R24.2
- no-connect marks 30 -> 28
Other:
- note added: "(VBATT while the latch is held or the button is"
- note added: "144 components / 91 nets / 4-layer JLCPCB stackup. Power rails (GND, 3V3, VBATT, VSYS, VLED, VBUS, VDD_CORE) are power symbols; only cross-block signals use global labels. Generated from scripts/circuit.py — do not hand-edit; rebuild with `python3 build.py --only schematic`."
- note added: "1M:1M divider off SW_ON, the power latch's output"
- note added: "3V3 LDO — EN = power latch OR USB (diode-OR, clamped)"
- note added: "J1 is a TYPE-C-31-M-12 right-angle receptacle. VBUS charges the cell AND (rev 2) runs"
- note added: "Latch / battery sense -> ADC"
- note added: "Li-ion charger (LGS4056H, 50mA) + LPR302823 LiPo"
- note added: "OFF + USB: reads 0, telling firmware to show charge"
- note added: "PWR_HOLD high so Q5 keeps LATCH_G low after release. Long press:"
- note added: "Press: BTN_N -> GND pulls LATCH_G low through D4 A2, Q4 turns on,"
- note added: "R17's pulldown EN sits at ~VBUS/2, and D2's second diode"
- note added: "Rev 2: USB boots the board even with the latch off. Against"
- note added: "SILICON (BAV70W), not Schottky: A1's reverse leak x R24 must stay"
- note added: "SW_ON = VBATT enables the LDO through D2. The CPU then drives"
- note added: "SW_ON=0 on the sense divider and shows charge status"
- note added: "With the board off, BTN_N sits near VBATT, so A1 is"
- note added: "clamps it to VBATT+Vf (NCP730 abs max V_EN is VIN+0.3, even"
- note added: "during precharge of a dead cell). Firmware then sees"
- note added: "firmware drops PWR_HOLD and power falls when the button is"
- note added: "instead of running the show."
- note added: "power button + soft latch"
- note added: "pressed). Latch ON: VBATT/2 battery telemetry. Latch"
- note added: "released. BTN_SENSE (pull-up) reads the button through D4 A1."
- note added: "reverse-biased and nothing reaches the unpowered pin. D4 is"
- note added: "status instead of running the show. GPIO29/ADC3."
- note added: "the board through D3 -> VSYS while a cable is in — see the power-path block."
- note added: "under Q4's 0.45V minimum threshold even hot, and a BAT54 leaks"
- note added: "~20uA at 85C. C27 = ESD/debounce on the edge button."
- note removed: "138 components / 87 nets / 4-layer JLCPCB stackup. Power rails (GND, 3V3, VBATT, VSYS, VLED, VBUS, VDD_CORE) are power symbols; only cross-block signals use global labels. Generated from scripts/circuit.py — do not hand-edit; rebuild with `python3 build.py --only schematic`."
- note removed: "1M:1M divider off SW_ON, the switch common (rev 2 — was"
- note removed: "3V3 LDO — EN = slide switch OR USB (diode-OR, clamped)"
- note removed: "J1 is a TYPE-C-31-M-12 right-angle receptacle. VBUS is charge-only: there is no"
- note removed: "Li-ion charger (LGS4056H, ~41mA) + RJD2032C1 cell"
- note removed: "Rev 2: USB boots the board even with SW2 off. Against R17's"
- note removed: "Switch / battery sense -> ADC"
- note removed: "Switch OFF + USB: reads 0, telling firmware to show"
- note removed: "VBATT). Switch ON: VBATT/2 battery telemetry as before."
- note removed: "VBUS->3V3 path, the MCU always runs from the cell."
- note removed: "charge status instead of running the show. GPIO29/ADC3."
- note removed: "it to VBATT+Vf (NCP730 abs max V_EN is VIN+0.3, even during"
- note removed: "precharge of a dead cell). Firmware then sees SW_ON=0 on"
- note removed: "pulldown EN sits at ~VBUS/2, and D2's second diode clamps"
- note removed: "running the show."
- note removed: "the sense divider and shows charge status instead of"
- moved on the sheet: C11, C12, C13, C14, C15, C22, C25, C5, C6, L1, R1, R13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

Commit message: One-button BOOTSEL, silicon D2/D3, button TVS, high-Vth latch FET
Folds the power-button simulation's findings into the board (user decisions
2026-10-24), each re-simulated, independently reviewed and re-reviewed.

- SW1 deleted. A long hold on the power button resets the chip into BOOTSEL
  (Q8/R26/R27, R28 680k + C75 timer, D5, U8 74LVC2G14GW, Q7 strap, C76/R29 ->
  Q6 RUN kick, C77). Fires 2.2-10.3 s typical, 2.0-19.4 s at U8's leakage
  limit. On battery the same hold turns the board off on release, which is
  the hardware force-off for hung firmware. Flash is never touched.
- Hot self-start fixed: D2 BAT54SW -> BAV99W, D3 B5819WS -> 1N4007WS. Board-off
  EN is now <= 0.03 V at 85 C (afabd86 reached 2.27 V). Cost: VSYS = VBUS - 0.8 V.
- Button ESD: D6 PESD5V0S1BL at the switch pad + R30 1k. A +-8 kV strike puts
  <= 22 mA into the latch (was ~24 A) and no longer counts as a press.
- Q4 CJ2101 -> LBSS84WT1G (VGS(th) 0.8-2.0 V): the latch's hot off-state
  margin no longer depends on an unspecified threshold tempco (review F2;
  design/sim/button/leakstudy.py).
- D4 BAV70W sourced from Nexperia (the Diodes part was down to 100 in stock).
- Testbench: netlist from circuit.py, afabd86 kept as a reference patch,
  54/54 runs pass, ESD/II-limit/pull-up/click-then-hold scenarios added.
- Placement: 14 new parts via scan_spot (12 back, Q6/R29 front in SW1's
  spot); DRC 0 errors, placed but NOT routed. Schematic regenerated
  (97 nets verified). Gates 1/2/6/8 updated with both reviews.

Firmware must change with this board: GPIO21 is active high with no pull-up,
and the long-press-off must be <= 1.5 s.

Co-Authored-By: Claude Opus 5.5 <noreply@anthropic.com>
Parts:
- removed SW1: BOOTSEL, earring:KEY-SMD_4P-L4.2-W3.2-P2.20-LS4.6, symbol gen:SW_PUSH
- added C75: 10u, earring:C_0603_1608Metric, symbol gen:C
- added C76: 10n, earring:C_0402_1005Metric, symbol gen:C
- added C77: 100n, earring:C_0402_1005Metric, symbol gen:C
- added D5: 1N4148WS, earring:D_SOD-323, symbol gen:D
- added D6: PESD5V0S1BL, earring:D_SOD-882, symbol gen:D_TVS
- added Q6, Q7: BSS138W, earring:SOT-323_MOSFET, symbol gen:Q_NMOS
- added Q8: CJ2101, earring:SOT-323_MOSFET, symbol gen:Q_PMOS_HS
- added R26: 100k, earring:R_0402_1005Metric, symbol gen:R
- added R27: 4.7k, earring:R_0402_1005Metric, symbol gen:R
- added R28: 680k, earring:R_0402_1005Metric, symbol gen:R
- added R29: 1M, earring:R_0402_1005Metric, symbol gen:R
- added R30: 1k, earring:R_0402_1005Metric, symbol gen:R
- added U8: 74LVC2G14, earring:SOT-363_SC-70-6, symbol gen:logic_schmitt2
- D2: value BAT54S -> BAV99W
- D3: value B5819WS -> 1N4007WS; symbol gen:D_SCH -> gen:D
- Q4: value CJ2101 -> LBSS84WT1G
Connections:
- net 3V3: now also C77.1, Q8.2 (S), R26.1, U8.5 (VCC)
- net BOOTSEL_SW: now also Q7.3 (D)
- net BTN_N: now also R30.2; no longer SW2.2
- net BTN_SENSE: now also D5.1 (K), Q8.3 (D), R27.1, R28.1; no longer D4.1 (A1)
- net GND: now also C75.2, C77.2, D6.2, Q6.2 (S), Q7.2 (S), R27.2, R29.2, U8.2 (GND)
- net RUN: now also Q6.3 (D)
- new net BOOT_TMR: C75.1, D5.2 (A), R28.2, U8.1 (1A)
- new net BTN_EXT: D6.1, R30.1, SW2.2
- new net LONG: C76.1, Q7.1 (G), U8.4 (2Y)
- new net LONG_N: U8.3 (2A), U8.6 (1Y)
- new net PRESS_N: D4.1 (A1), Q8.1 (G), R26.2
- new net RUN_KICK: C76.2, Q6.1 (G), R29.1
- no-connect marks 28 -> 26
Other:
- note added: "(power-button long hold) pulls BOOTSEL_SW low."
- note added: "157 components / 97 nets / 4-layer JLCPCB stackup. Power rails (GND, 3V3, VBATT, VSYS, VLED, VBUS, VDD_CORE) are power symbols; only cross-block signals use global labels. Generated from scripts/circuit.py — do not hand-edit; rebuild with `python3 build.py --only schematic`."
- note added: "Hold the power button: BTN_SENSE goes high (Q8), C75 charges through R28 and U8 trips 2.2-10.3s later (5s typ; spread"
- note added: "Pico-style: QSPI_SS is both the flash /CS and the BOOTSEL strap. Q7"
- note added: "SILICON (BAV70W), not Schottky: the off-state leaks x R24 must"
- note added: "a strike at the pad and R30 keeps it off BTN_N/D4; C27 debounces."
- note added: "block turns that into BTN_SENSE). With the board off BTN_N sits"
- note added: "empties C75 on release. Firmware: GPIO21 no pull-up, high = held; long-press-off < 2s."
- note added: "is U8's VT+ and C75's X5R tolerance/bias, simulated in design/sim/button). LONG straps QSPI_SS low through Q7/R3 for as"
- note added: "long as the button is held and kicks RUN low for ~10ms (C76/R29 -> Q6): the chip resets into BOOTSEL. Flash is not"
- note added: "near VBATT and PRESS_N at 0V, so A1 is reverse-biased. D4 is"
- note added: "one button: long hold = BOOTSEL / force-off"
- note added: "released. D4 A1 pulls PRESS_N low while pressed (the one-button"
- note added: "stay under Q4's 0.45V minimum threshold even hot. ESD: D6 clamps"
- note added: "touched. On battery the reset drops PWR_HOLD, so the board turns off on release: the force-off for hung firmware. D5"
- note removed: "144 components / 91 nets / 4-layer JLCPCB stackup. Power rails (GND, 3V3, VBATT, VSYS, VLED, VBUS, VDD_CORE) are power symbols; only cross-block signals use global labels. Generated from scripts/circuit.py — do not hand-edit; rebuild with `python3 build.py --only schematic`."
- note removed: "Pico-style: QSPI_SS is both the flash /CS and the BOOTSEL strap."
- note removed: "SILICON (BAV70W), not Schottky: A1's reverse leak x R24 must stay"
- note removed: "With the board off, BTN_N sits near VBATT, so A1 is"
- note removed: "released. BTN_SENSE (pull-up) reads the button through D4 A1."
- note removed: "reverse-biased and nothing reaches the unpowered pin. D4 is"
- note removed: "under Q4's 0.45V minimum threshold even hot, and a BAT54 leaks"
- note removed: "~20uA at 85C. C27 = ESD/debounce on the edge button."
- moved on the sheet: SW2

Commit message: LED ring: WS2816C-1313 (16-bit) in three switched zones; lock policy
User decisions 2026-10-24: switch the ring to WS2816C-1313/4P and split it
into left / right / centre zones. Independently reviewed (gates 1, 2, 6 pass).

- LEDs: SK6805-EC10 -> WS2816C-1313/4P (C42417612). 16-bit per channel plus
  gamma for the low-brightness range; VDD floor 3.3 V; idle 0.7-1.0 mA per LED;
  rated to 65 C; MSL 5a. New LED_WS2816C-1313 footprint (EasyEDA land, pin map
  checked against the datasheet: 1 VDD, 2 DO, 3 GND, 4 DI).
- Three zones, each its own chain, TPS22913 load switch (U4/U9/U10) and
  open-drain shifter pulled up to its own rail (Q3/Q9/Q10 + R23/R31/R32), so a
  dark zone draws nothing and can't be back-fed through its data line.
  Left LED1-18, right LED37->19 (reversed, enters at the tip), centre
  LED38-45. Data GPIO16/17/18 (adjacent: one PIO program), enables GPIO1/0/22.
- In2: VLED_C inner band, VLED_L / VLED_R split of the outer band, 3V3 disc.
- Placement: same ring centres, per-zone orientation; D3/C29 moved for
  LED44; zone drivers via scan_spot. DRC 0 errors, placed but NOT routed:
  the user routes it with their own GPU autorouter. route.py's SK6805-era
  freerouting workaround pre-routes are removed.
- Locked for the router: all LEDs, J1, SW2 (user request), plus BT1, Q1, and
  every part that locked copper or a fixed pour lands on (U1, U2, U5, R14,
  VREG cluster L1/C11/C12/C13/R13/C22). Everything else may be nudged.
- Schematic regenerated per zone (103 nets verified).

Firmware: three 48-bit chains (reset >= 280 us), data pins inverted and idle
high, power zones off rather than blanking them, keep a hard brightness cap.

Co-Authored-By: Claude Opus 5.5 <noreply@anthropic.com>
Parts:
- added C78, C79: 10u, earring:C_0603_1608Metric, symbol gen:C
- added Q10, Q9: BSS138W, earring:SOT-323_MOSFET, symbol gen:Q_NMOS
- added R31, R32: 1k, earring:R_0402_1005Metric, symbol gen:R
- added R33, R34: 10k, earring:R_0402_1005Metric, symbol gen:R
- added U10, U9: TPS22913, earring:YZV0004ADAD, symbol gen:load_switch
- LED1, LED10, LED11, LED12, LED13, LED14, LED15, LED16, LED17, LED18, LED19, LED2, LED20, LED21, LED22, LED23, LED24, LED25, LED26, LED27, LED28, LED29, LED3, LED30, LED31, LED32, LED33, LED34, LED35, LED36, LED37, LED38, LED39, LED4, LED40, LED41, LED42, LED43, LED44, LED45, LED5, LED6, LED7, LED8, LED9: value SK6805-EC10 -> WS2816C-1313; footprint earring:LED_SK6805-EC10 -> earring:LED_WS2816C-1313
Connections:
- net GND: now also LED1.3 (GND), LED10.3 (GND), LED11.3 (GND), LED12.3 (GND), LED13.3 (GND), LED14.3 (GND), LED15.3 (GND), LED16.3 (GND), LED17.3 (GND), LED18.3 (GND), LED19.3 (GND), LED2.3 (GND), LED20.3 (GND), LED21.3 (GND), LED22.3 (GND), LED23.3 (GND), LED24.3 (GND), LED25.3 (GND), LED26.3 (GND), LED27.3 (GND), LED28.3 (GND), LED29.3 (GND), LED3.3 (GND), LED30.3 (GND), LED31.3 (GND), LED32.3 (GND), LED33.3 (GND), LED34.3 (GND), LED35.3 (GND), LED36.3 (GND), LED37.3 (GND), LED38.3 (GND), LED39.3 (GND), LED4.3 (GND), LED40.3 (GND), LED41.3 (GND), LED42.3 (GND), LED43.3 (GND), LED44.3 (GND), LED45.3 (GND), LED5.3 (GND), LED6.3 (GND), LED7.3 (GND), LED8.3 (GND), LED9.3 (GND), C78.2, C79.2, Q10.2 (S), Q9.2 (S), R33.2, R34.2, U10.B1 (GND), U9.B1 (GND); no longer LED1.1 (GND), LED10.1 (GND), LED11.1 (GND), LED12.1 (GND), LED13.1 (GND), LED14.1 (GND), LED15.1 (GND), LED16.1 (GND), LED17.1 (GND), LED18.1 (GND), LED19.1 (GND), LED2.1 (GND), LED20.1 (GND), LED21.1 (GND), LED22.1 (GND), LED23.1 (GND), LED24.1 (GND), LED25.1 (GND), LED26.1 (GND), LED27.1 (GND), LED28.1 (GND), LED29.1 (GND), LED3.1 (GND), LED30.1 (GND), LED31.1 (GND), LED32.1 (GND), LED33.1 (GND), LED34.1 (GND), LED35.1 (GND), LED36.1 (GND), LED37.1 (GND), LED38.1 (GND), LED39.1 (GND), LED4.1 (GND), LED40.1 (GND), LED41.1 (GND), LED42.1 (GND), LED43.1 (GND), LED44.1 (GND), LED45.1 (GND), LED5.1 (GND), LED6.1 (GND), LED7.1 (GND), LED8.1 (GND), LED9.1 (GND)
- net VSYS: now also U10.A2 (VIN), U9.A2 (VIN)
- net LED_EN_R: now reaches U1.2 (GPIO0)
- net LED_EN_R: now also R33.1, U9.B2 (ON)
- net LED_DATA_C: now reaches U1.27 (GPIO16)
- net LED_DATA_C: now also Q10.1 (G)
- net LED_DATA_R: now reaches U1.28 (GPIO17)
- net LED_DATA_R: now also Q9.1 (G)
- net LED_EN_C: now reaches U1.34 (GPIO22)
- net LED_EN_C: now also R34.1, U10.B2 (ON)
- net LEDC_D7: now reaches LED45.4 (DI)
- net LEDC_D7: now also LED44.2 (DO)
- net LED_D0 renamed LEDL_D0
- net LEDL_D0: now also LED1.4 (DI); no longer LED1.2 (DI)
- net LED_D1 renamed LEDL_D2
- net LEDL_D2: now also LED3.4 (DI); no longer LED1.4 (DO)
- net LED_D10 renamed LEDL_D11
- net LEDL_D11: now also LED12.4 (DI); no longer LED10.4 (DO)
- net LED_D11 renamed LEDL_D10
- net LEDL_D10: now also LED10.2 (DO); no longer LED12.2 (DI)
- net LED_D12 renamed LEDL_D13
- net LEDL_D13: now also LED14.4 (DI); no longer LED12.4 (DO)
- net LED_D13 renamed LEDL_D12
- net LEDL_D12: now also LED12.2 (DO); no longer LED14.2 (DI)
- net LED_D14 renamed LEDL_D15
- net LEDL_D15: now also LED16.4 (DI); no longer LED14.4 (DO)
- net LED_D15 renamed LEDL_D14
- net LEDL_D14: now also LED14.2 (DO); no longer LED16.2 (DI)
- net LED_D16 renamed LEDL_D17
- net LEDL_D17: now also LED18.4 (DI); no longer LED16.4 (DO)
- net LED_D17: no longer names the net of LED18.2 (DO)
- net LED_D17: no longer LED17.4 (DO)
- net LED_D18: no longer names the net of LED19.2 (DO)
- net LED_D18: no longer LED18.4 (DO)
- net LED_D19 renamed LEDR_D18
- net LED_D2 renamed LEDL_D1
- net LEDL_D1: now also LED1.2 (DO); no longer LED3.2 (DI)
- net LED_D20 renamed LEDR_D17
- net LED_D21 renamed LEDR_D16
- net LED_D22 renamed LEDR_D15
- net LED_D23 renamed LEDR_D14
- net LED_D24 renamed LEDR_D13
- net LED_D25 renamed LEDR_D12
- net LED_D26 renamed LEDR_D11
- net LED_D27 renamed LEDR_D10
- net LED_D28 renamed LEDR_D9
- net LED_D29 renamed LEDR_D8
- net LED_D3 renamed LEDL_D4
- net LEDL_D4: now also LED5.4 (DI); no longer LED3.4 (DO)
- net LED_D30 renamed LEDR_D7
- net LED_D31 renamed LEDR_D6
- net LED_D32 renamed LEDR_D5
- net LED_D33 renamed LEDR_D4
- net LED_D34 renamed LEDR_D3
- net LED_D35 renamed LEDR_D2
- net LED_D36 renamed LEDR_D1
- net LED_D37 renamed LEDC_D1
- net LEDC_D1: now also LED39.4 (DI); no longer LED37.4 (DO)
- net LED_D38 renamed LEDC_D0
- net LEDC_D0: now also Q10.3 (D), R32.2; no longer LED39.2 (DI)
- net LED_D39 renamed LEDC_D3
- net LEDC_D3: now also LED41.4 (DI); no longer LED39.4 (DO)
- net LED_D4 renamed LEDL_D3
- net LEDL_D3: now also LED3.2 (DO); no longer LED5.2 (DI)
- net LED_D40 renamed LEDC_D2
- net LEDC_D2: now also LED39.2 (DO); no longer LED41.2 (DI)
- net LED_D41 renamed LEDC_D5
- net LEDC_D5: now also LED43.4 (DI); no longer LED41.4 (DO)
- net LED_D42 renamed LEDC_D4
- net LEDC_D4: now also LED41.2 (DO); no longer LED43.2 (DI)
- removed net LED_D43: LED43.4 (DO), LED44.2 (DI)
- net LED_D44: no longer names the net of LED45.2 (DO)
- net LED_D44: no longer LED44.4 (DO)
- net LED_D5 renamed LEDL_D6
- net LEDL_D6: now also LED7.4 (DI); no longer LED5.4 (DO)
- net LED_D6 renamed LEDL_D5
- net LEDL_D5: now also LED5.2 (DO); no longer LED7.2 (DI)
- net LED_D7 renamed LEDL_D8
- net LEDL_D8: now also LED9.4 (DI); no longer LED7.4 (DO)
- net LED_D8 renamed LEDL_D7
- net LEDL_D7: now also LED7.2 (DO); no longer LED9.2 (DI)
- removed net LED_D9: LED10.2 (DI), LED9.4 (DO)
- net LED_DATA renamed LED_DATA_L
- net LED_EN renamed LED_EN_L
- removed net VLED: C20.1, C30.1, C32.1, C34.1, C36.1, C38.1, C40.1, C42.1, C44.1, C46.1, C48.1, C50.1, C52.1, C54.1, C56.1, C58.1, C60.1, C62.1, C64.1, C66.1, C68.1, C70.1, C72.1, C74.1, LED1.3 (VDD), LED10.3 (VDD), LED11.3 (VDD), LED12.3 (VDD), LED13.3 (VDD), LED14.3 (VDD), LED15.3 (VDD), LED16.3 (VDD), LED17.3 (VDD), LED18.3 (VDD), LED19.3 (VDD), LED2.3 (VDD), LED20.3 (VDD), LED21.3 (VDD), LED22.3 (VDD), LED23.3 (VDD), LED24.3 (VDD), LED25.3 (VDD), LED26.3 (VDD), LED27.3 (VDD), LED28.3 (VDD), LED29.3 (VDD), LED3.3 (VDD), LED30.3 (VDD), LED31.3 (VDD), LED32.3 (VDD), LED33.3 (VDD), LED34.3 (VDD), LED35.3 (VDD), LED36.3 (VDD), LED37.3 (VDD), LED38.3 (VDD), LED39.3 (VDD), LED4.3 (VDD), LED40.3 (VDD), LED41.3 (VDD), LED42.3 (VDD), LED43.3 (VDD), LED44.3 (VDD), LED45.3 (VDD), LED5.3 (VDD), LED6.3 (VDD), LED7.3 (VDD), LED8.3 (VDD), LED9.3 (VDD), R23.1, U4.A1 (VOUT)
- new net LEDC_D6: LED43.2 (DO), LED44.4 (DI)
- new net LEDL_D16: LED16.2 (DO), LED17.4 (DI)
- new net LEDL_D9: LED10.4 (DI), LED9.2 (DO)
- new net LEDR_D0: LED37.4 (DI), Q9.3 (D), R31.2
- new net VLED_C: C68.1, C70.1, C72.1, C74.1, C79.1, LED38.1 (VDD), LED39.1 (VDD), LED40.1 (VDD), LED41.1 (VDD), LED42.1 (VDD), LED43.1 (VDD), LED44.1 (VDD), LED45.1 (VDD), R32.1, U10.A1 (VOUT)
- new net VLED_L: C20.1, C30.1, C32.1, C34.1, C36.1, C38.1, C40.1, C42.1, C44.1, C46.1, LED1.1 (VDD), LED10.1 (VDD), LED11.1 (VDD), LED12.1 (VDD), LED13.1 (VDD), LED14.1 (VDD), LED15.1 (VDD), LED16.1 (VDD), LED17.1 (VDD), LED18.1 (VDD), LED2.1 (VDD), LED3.1 (VDD), LED4.1 (VDD), LED5.1 (VDD), LED6.1 (VDD), LED7.1 (VDD), LED8.1 (VDD), LED9.1 (VDD), R23.1, U4.A1 (VOUT)
- new net VLED_R: C48.1, C50.1, C52.1, C54.1, C56.1, C58.1, C60.1, C62.1, C64.1, C66.1, C78.1, LED19.1 (VDD), LED20.1 (VDD), LED21.1 (VDD), LED22.1 (VDD), LED23.1 (VDD), LED24.1 (VDD), LED25.1 (VDD), LED26.1 (VDD), LED27.1 (VDD), LED28.1 (VDD), LED29.1 (VDD), LED30.1 (VDD), LED31.1 (VDD), LED32.1 (VDD), LED33.1 (VDD), LED34.1 (VDD), LED35.1 (VDD), LED36.1 (VDD), LED37.1 (VDD), R31.1, U9.A1 (VOUT)
- no-connect marks 26 -> 24
Other:
- note added: "167 components / 103 nets / 4-layer JLCPCB stackup. Power rails (GND, 3V3, VBATT, VSYS, VLED, VBUS, VDD_CORE) are power symbols; only cross-block signals use global labels. Generated from scripts/circuit.py — do not hand-edit; rebuild with `python3 build.py --only schematic`."
- note added: "Addressable LED ring — 45 x WS2816C-1313 in three zone chains"
- note added: "GPIO16/17/18; one PIO program can clock all three consecutive pins."
- note added: "LED bypass, centre zone — 100n VLED_C-GND, one per two LEDs"
- note added: "LED bypass, left zone — 100n VLED_L-GND, one per two LEDs"
- note added: "LED bypass, right zone — 100n VLED_R-GND, one per two LEDs"
- note added: "LED data level shifters — one open-drain stage per zone"
- note added: "One switch per zone: the WS2816C idles at 0.7-1.0mA per LED, so only lit"
- note added: "Three independent chains, each with its own switched rail: left LED1->LED18, right LED37->LED19 (entering at the tip chevron), centre LED38->LED45. A dark zone is unpowered, so data never crosses a zone boundary; each row break carries on through LED<z>_D<n>."
- note added: "VLED zone load switches (dark zones draw zero)"
- note added: "WS2816C VIH is 0.7*VDD: 2.94V on a full cell, 3.47V on a 5.25V port, above a 3.3V pad, so each zone's first pixel is"
- note added: "driven through an open-drain inverter into a 1k pull-up on THAT zone's rail. A dark zone's pull-up is dead, so its"
- note added: "first DI is never driven into an unpowered LED. Firmware: gpio_set_outover(pin, GPIO_OVERRIDE_INVERT) on"
- note added: "its LED_EN high."
- note added: "next to their LEDs around the ring"
- note added: "zones are powered. The pull-downs hold every zone off until firmware drives"
- note removed: "157 components / 97 nets / 4-layer JLCPCB stackup. Power rails (GND, 3V3, VBATT, VSYS, VLED, VBUS, VDD_CORE) are power symbols; only cross-block signals use global labels. Generated from scripts/circuit.py — do not hand-edit; rebuild with `python3 build.py --only schematic`."
- note removed: "Addressable LED ring — 45 x SK6805-EC10 daisy chain"
- note removed: "C30..C74, distributed around the ring next to their LEDs"
- note removed: "Chain runs LED1 -> LED45 in board order; each row break carries on through LED_D<n>. VLED is the switched battery rail, so the ring is dark until LED_EN goes high."
- note removed: "LED data level shifter — open-drain into the ring"
- note removed: "LED ring bypass — 100n VLED-GND, one per two LEDs"
- note removed: "R10 holds the switch off until firmware drives LED_EN high."
- note removed: "The ring's VIH is 0.7*VLED. On the cell that peaked at 2.94V and the MCU drove pixel 1"
- note removed: "VLED high-side load switch (LEDs draw zero when off)"
- note removed: "directly; on VSYS it is 3.29V (3.5V at a 5.25V port), past anything a 3.3V pad can"
- note removed: "output. Q3 inverts into R23's pull-up, so the swing is a full VLED rail whatever VLED is"
- note removed: "override sits after the PIO, so the NeoPixel program is untouched."
- note removed: "previous DO. Firmware must set gpio_set_outover(LED_DATA, GPIO_OVERRIDE_INVERT) — the pad"
- note removed: "— 3.0V cell or 5.0V cable. Only pixel 1 needs it; every DI after that is driven by the"
- moved on the sheet: C11, C12, C13, C14, C15, C20, C22, C25, C30, C32, C34, C36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
